Commit message: gazebo

File: description/gazebo_control.xacro (robot description, xacro)
@@ -19,3 +19,22 @@
         </plugin>
     </gazebo>
+<link name="imu_link"/>
+<joint name="imu_joint" type="fixed">
+  <parent link="base_link"/>
+  <child link="imu_link"/>
+  <origin xyz="0 0 0.1" rpy="0 0 0"/>
+</joint>
+<gazebo reference="imu_link">
+  <sensor name="imu_sensor" type="imu">
+    <always_on>true</always_on>
+    <update_rate>50</update_rate>
+    <plugin name="imu_plugin" filename="libgazebo_ros_imu_sensor.so">
+      <ros>
+        <namespace>/</namespace>
+      </ros>
+      <frame_name>imu_link</frame_name>
+      <topic_name>/imu</topic_name>
+    </plugin>
+  </sensor>
+</gazebo>
 </robot>

Commit message: remove error

File: description/gazebo_control.xacro (robot description, xacro)
@@ -19,22 +19,3 @@
         </plugin>
     </gazebo>
-<link name="imu_link"/>
-<joint name="imu_joint" type="fixed">
-  <parent link="base_link"/>
-  <child link="imu_link"/>
-  <origin xyz="0 0 0.1" rpy="0 0 0"/>
-</joint>
-<gazebo reference="imu_link">
-  <sensor name="imu_sensor" type="imu">
-    <always_on>true</always_on>
-    <update_rate>50</update_rate>
-    <plugin name="imu_plugin" filename="libgazebo_ros_imu_sensor.so">
-      <ros>
-        <namespace>/</namespace>
-      </ros>
-      <frame_name>imu_link</frame_name>
-      <topic_name>/imu</topic_name>
-    </plugin>
-  </sensor>
-</gazebo>
 </robot>
