Commit message: ب

File: description/robot_core.xacro (robot description, xacro)
@@ -126,3 +126,37 @@
         <mu2 value="0.001"/>
     </gazebo>
+    <!-- IMU sensor -->
+<gazebo>
+  <sensor name="imu_sensor" type="imu">
+    <always_on>true</always_on>
+    <update_rate>50</update_rate>
+    <imu>
+      <noise>
+        <type>gaussian</type>
+        <rate>
+          <mean>0.0</mean>
+          <stddev>0.001</stddev>
+        </rate>
+        <accel>
+          <mean>0.0</mean>
+          <stddev>0.1</stddev>
+        </accel>
+      </noise>
+    </imu>
+    <plugin name="imu_plugin" filename="libgazebo_ros_imu_sensor.so">
+      <ros>
+        <namespace>/</namespace>
+        <remapping>~/out:=/imu</remapping>
+      </ros>
+      <frame_name>imu_link</frame_name>
+    </plugin>
+  </sensor>
+</gazebo>
+<link name="imu_link">
+</link>
+<joint name="imu_joint" type="fixed">
+  <parent link="base_link"/>
+  <child link="imu_link"/>
+  <origin xyz="0 0 0.1" rpy="0 0 0"/>
+</joint>
 </robot>

Commit message: IMU sensor

File: description/robot_core.xacro (robot description, xacro)
@@ -153,4 +153,25 @@
   </sensor>
 </gazebo>
+<!-- IMU START -->
+<link name="imu_link"/>
+<joint IMUname="imu_joint" type="fixed">
+  <parent link="base_link"/>
+  <child link="imu_link"/>
+  <origin xyz="0 0 0.1" rpy="0 0 0"/>
+</joint>
+<gazebo reference="imu_link">
+  <sensor name="imu_sensor" type="imu">
+    <update_rate>50</update_rate>
+    <always_on>true</always_on>
+    <plugin name="imu_plugin" filename="libgazebo_ros_imu_sensor.so">
+      <ros>
+        <namespace>/</namespace>
+      </ros>
+      <frame_name>imu_link</frame_name>
+      <topic_name>/imu</topic_name>
+    </plugin>
+  </sensor>
+</gazebo>
+<!-- IMU END -->
 <link name="imu_link">
 </link>

Commit message: remove IMU

File: description/robot_core.xacro (robot description, xacro)
@@ -126,58 +126,3 @@
         <mu2 value="0.001"/>
     </gazebo>
-    <!-- IMU sensor -->
-<gazebo>
-  <sensor name="imu_sensor" type="imu">
-    <always_on>true</always_on>
-    <update_rate>50</update_rate>
-    <imu>
-      <noise>
-        <type>gaussian</type>
-        <rate>
-          <mean>0.0</mean>
-          <stddev>0.001</stddev>
-        </rate>
-        <accel>
-          <mean>0.0</mean>
-          <stddev>0.1</stddev>
-        </accel>
-      </noise>
-    </imu>
-    <plugin name="imu_plugin" filename="libgazebo_ros_imu_sensor.so">
-      <ros>
-        <namespace>/</namespace>
-        <remapping>~/out:=/imu</remapping>
-      </ros>
-      <frame_name>imu_link</frame_name>
-    </plugin>
-  </sensor>
-</gazebo>
-<!-- IMU START -->
-<link name="imu_link"/>
-<joint IMUname="imu_joint" type="fixed">
-  <parent link="base_link"/>
-  <child link="imu_link"/>
-  <origin xyz="0 0 0.1" rpy="0 0 0"/>
-</joint>
-<gazebo reference="imu_link">
-  <sensor name="imu_sensor" type="imu">
-    <update_rate>50</update_rate>
-    <always_on>true</always_on>
-    <plugin name="imu_plugin" filename="libgazebo_ros_imu_sensor.so">
-      <ros>
-        <namespace>/</namespace>
-      </ros>
-      <frame_name>imu_link</frame_name>
-      <topic_name>/imu</topic_name>
-    </plugin>
-  </sensor>
-</gazebo>
-<!-- IMU END -->
-<link name="imu_link">
-</link>
-<joint name="imu_joint" type="fixed">
-  <parent link="base_link"/>
-  <child link="imu_link"/>
-  <origin xyz="0 0 0.1" rpy="0 0 0"/>
-</joint>
 </robot>
